File: PCB/cap/cap.sch (KiCad schematic (older format))
At the start: 14 parts, among them J1 Servo1, J2 Servo2, J3 LimitSwitchA, J4 Conn_01x02_Female, J5 Conn_01x02_Female, J6 LimitSwitchB, J7 Conn_01x02_Female

Commit message: Add current sensor and rename project to follow software branch.
Parts:
- added D?: D_Zener, symbol Device:D_Zener
- added R? (x3): ?, symbol Device:R
- added U?: ZXCT1009F, Package_TO_SOT_SMD:SOT-23, symbol Amplifier_Current:ZXCT1009F
Connections:
- net labels added: +5VA, A2
- wire segments 59 -> 75
Other:
- note added: "Current Sensor"
- note added: "Larger surface mounted components\nResistor values for LEDs\nMounting holes on board\nDoes the RC need capacitor across power?\nCorrect foot prints?\n - 90 degree -> Servo\n - Screw terminal -> FSR\n"
- note added: "Measure new servos and then select a unit with correct full scale range."
- note added: "Radio"
- note removed: "Larger surface mounted components\nResistor values for LEDs\nMounting holes on board\nCorrect foot prints?\n - 90 degree -> Servo\n - Screw terminal -> FSR\n"
- moved on the sheet: A1
