File: PCB/vibration/vibration.sch (KiCad schematic (older format))
At the start: 16 parts, among them J1 Conn_01x02, J2 Conn_01x04, J3 Conn_01x02, U1 NRF24L01_Breakout, U2 LM7805

Commit message: minor tweaks and added completed vibration board - schematic and routing
Parts:
- removed C1: 0.22 uF, Capacitor_SMD:C_0603_1608Metric_Pad1.05x0.95mm_HandSolder, symbol Device:C
- removed C2: 0.1 uF, Capacitor_SMD:C_0603_1608Metric_Pad1.05x0.95mm_HandSolder, symbol Device:C
- removed J2: Conn_01x04, Connector_Molex:Molex_Micro-Fit_3.0_43650-0400_1x04_P3.00mm_Horizontal, symbol Connector_Generic:Conn_01x04
- removed J3: Conn_01x02, Connector_Molex:Molex_Micro-Fit_3.0_43650-0200_1x02_P3.00mm_Horizontal, symbol Connector_Generic:Conn_01x02
- removed U2: LM7805, Package_TO_SOT_SMD:SOT-223-3_TabPin2, symbol Regulator_Linear:LM7805_TO220
- added J2, J3: Conn_01x03, Connector_Molex:Molex_Micro-Fit_3.0_43650-0300_1x03_P3.00mm_Horizontal, symbol Connector_Generic:Conn_01x03
- added J4, J5: Conn_01x04, Connector_Molex:Molex_Micro-Fit_3.0_43650-0400_1x04_P3.00mm_Horizontal, symbol Connector_Generic:Conn_01x04
- added Q1, Q2: BSS138, Package_TO_SOT_SMD:SOT-23, symbol Transistor_FET:BSS138
- added R3, R4, R5, R6: 10 kOhm, Resistor_SMD:R_0603_1608Metric_Pad1.05x0.95mm_HandSolder, symbol Device:R
Connections:
- net labels added: D4, SCL, SDA
- net labels removed: D6, Vdrive
- wire segments 53 -> 77
Other:
- note added: "Aux"
- note added: "I2C 3.3 Logic"
- note added: "I2C 5.0 Logic"
- note removed: "Camera Power"
- note removed: "PWM Control"
- note removed: "To be mated with Digi-Key part numbers:\nH2184-ND‎\nH4BXT-10106-B8-ND"

Commit message: All schematics detail check complete
Other:
- note added: "Future Auxiliary Ports"
- note added: "Indicators"
- note added: "RF Communication"
- note removed: "Aux"
- note removed: "Communication"
- moved on the sheet: A1, J2, J3, J4, J5, Q1, Q2, R3, R4, R5, R6, U1
