File: PCB/camera/camera.sch (KiCad schematic (older format))
At the start: 16 parts, among them J1 Conn_01x02, J2 Conn_01x04, J3 Conn_01x02, U1 NRF24L01_Breakout, U2 LM7805

Commit message: All schematics detail check complete
Other:
- note added: "Indicators"
- note added: "RF Communication"
- note removed: "Communication"
- moved on the sheet: A1, C1, C2, J2, J3, U1, U2

Commit message: Camera review complete. Create gerbers
Connections:
- net D5: now also J2.4 (Pin_4); no longer J2.3 (Pin_3)
- net D6: now also J2.2 (Pin_2); no longer J2.1 (Pin_1)
- net GND: now also J2.1 (Pin_1), J2.3 (Pin_3); no longer J2.2 (Pin_2), J2.4 (Pin_4)
Changed lines of the file:
@@
-$EndComp
-$Comp
-L power:GND #PWR0110
-U 1 1 5EB4BBA3
-P 8150 5300
-F 0 "#PWR0110" H 8150 5050 50  0001 C CNN
-F 1 "GND" H 8155 5127 50  0000 C CNN
-F 2 "" H 8150 5300 50  0001 C CNN
-F 3 "" H 8150 5300 50  0001 C CNN
-	1    8150 5300
-	1    0    0    -1
 $EndComp
 $Comp
 L power:GND #PWR0115
 U 1 1 5EB4C016
-P 8550 5500
-F 0 "#PWR0115" H 8550 5250 50  0001 C CNN
-F 1 "GND" H 8555 5327 50  0000 C CNN
-F 2 "" H 8550 5500 50  0001 C CNN
-F 3 "" H 8550 5500 50  0001 C CNN
-	1    8550 5500
-	1    0    0    -1
-$EndComp
-Text GLabel 8450 5400 0    50   Input ~ 0
+P 8400 5400
+F 0 "#PWR0115" H 8400 5150 50  0001 C CNN
+F 1 "GND" H 8405 5227 50  0000 C CNN
+F 2 "" H 8400 5400 50  0001 C CNN
+F 3 "" H 8400 5400 50  0001 C CNN
+	1    8400 5400
+	1    0    0    -1
+$EndComp
+Text GLabel 8700 5500 0    50   Input ~ 0
 D5
-Text GLabel 8050 5200 0    50   Input ~ 0
+Text GLabel 8350 5300 0    50   Input ~ 0
 D6
 Wire Wire Line
-	8450 5400 8700 5400
-Wire Wire Line
 	8050 5200 8700 5200
-Wire Wire Line
-	8150 5300 8700 5300
-Wire Wire Line
-	8700 5500 8550 5500
 $Comp
 L power:VCC #PWR0116
@@
 Text Notes 8050 5950 0    39   Italic 0
 To be mated with Digi-Key part numbers:\nH2184-ND‎\nH4BXT-10106-B8-ND
+$Comp
+L power:GND #PWR0110
+U 1 1 5EB4BBA3
+P 8050 5200
+F 0 "#PWR0110" H 8050 4950 50  0001 C CNN
+F 1 "GND" H 8055 5027 50  0000 C CNN
+F 2 "" H 8050 5200 50  0001 C CNN
+F 3 "" H 8050 5200 50  0001 C CNN
+	1    8050 5200
+	1    0    0    -1
+$EndComp
+Wire Wire Line
+	8400 5400 8700 5400
+Wire Wire Line
+	8350 5300 8700 5300
 $EndSCHEMATC
